Commit message: Modified DARPA files for running on Edgar Mine ROS bag.

File: cartographer_ros/urdf/DARPA.urdf (robot description, URDF)
Before this commit: robot cartographer_backpack_3d, 3 links, 2 joints
Joints:
- joint imu_link_joint: origin xyz=0 0 0 rpy=3.14 0 1.57 -> xyz=0 0 0 rpy=3.14 0 3.14
