Commit message: Got good results (faster loop closures) with 1 Horizontal Ouster (bag_gene.launch). Re-organized files into tunnel and urban folders.

File: cartographer_ros/urdf/urban/aerial_F450_rig.urdf (robot description, URDF)
Before this commit: robot cartographer_backpack_3d, 3 links, 2 joints
Joints:
- joint os1_link_joint: origin xyz=0 0 0 rpy=3.14 0 3.14 -> xyz=0 0 -0.03 rpy=3.14 0 3.14
