Commit message: bag_gene...launch, cartographer 3D with one horizontal Ouster now works well! Turned off online IMU extrinsics. Also detuned loop closure. Works with aerial bags and with full rig bags.

File: cartographer_ros/urdf/urban/gene_full_rig_2_ouster_2_rplidar_backup.urdf (robot description, URDF)
Before this commit: robot cartographer_backpack_3d, 5 links, 4 joints
Joints:
- joint imu_link_joint: origin xyz=0 0 0 rpy=3.14159265359 0 1.57079632679 -> xyz=0 0 0 rpy=3.14421064747 0 1.56503674026
