Commit message: Implemented horizontal RPLIDAR in 3D Cartographer, poor results. Nominally looked okay, but suffers poor loop local closures at times, and is catastrophic. Also not loop closing so drifts off to obliviion. Cannot corrext Z-axis drift.

File: cartographer_ros/urdf/urban/gene_FullRig_2_Ouster_2_RPLIDAR.urdf (robot description, URDF)
Before this commit: robot cartographer_backpack_3d, 5 links, 4 joints
Links:
- removed link laser
- added link rp_0; visual cylinder length=0.07 radius=0.05
- added link rp_1; visual cylinder length=0.07 radius=0.05
Joints:
- removed joint laser_link_joint
- added joint rp_0_link_joint: type fixed, parent base_link, child rp_0, origin xyz=0.000129 -0.00333 0.05768 rpy=0.0 0.0 3.14159
- added joint rp_1_link_joint: type fixed, parent base_link, child rp_1, origin xyz=0.0 0.17145 -0.060325 rpy=-1.5708 0.0 3.14159
