Commit message: Old changes from Fall 2019 semester project on tilting RPLIDAR S1.

File: cartographer_ros/urdf/urban/gene_F650.urdf (robot description, URDF)
Before this commit: robot cartographer_backpack_3d, 3 links, 2 joints
Links:
- added link servo; visual cylinder length=0.07 radius=0.05
Joints:
- added joint servo_link_joint: type fixed, parent base_link, child servo, origin xyz=0.15 0 0 rpy=0 0 0
